File: ADS1298/ADS1298.sch (KiCad schematic (older format))
At the start: 108 parts, among them IC1 ADS1298, IC2 ADuM6401, IC3 ADuM4401, IC4 ADM811, IC5 REF5025, IC6 OPA211, P1 ADS_Sensors, U2 TPS79230, U3 TPS79101, U4 TPS72325, U5 TPS60403, U6 CONN_ADS1298

Commit message: Updated ADS1298 project and KiCAD libraries and tools.
git-svn-id: http://opendous.googlecode.com/svn/trunk/Current_Designs@183 3806c4c6-82b1-11dd-ad27-0f66e57d2035
Parts:
- removed P1: ADS_Sensors, symbol CONN_20X2
- added P1: ADS_Sensors, symbol CONN_25X2
- added R22: 2.2, symbol R_MINI
Connections:
- wire segments 244 -> 253
- no-connect marks 13 -> 10
Other:
- note added: "2mm RA Header"
- moved on the sheet: TP2

Commit message: Updated ADS1298 project; added notes to schematic.
git-svn-id: http://opendous.googlecode.com/svn/trunk/Current_Designs@184 3806c4c6-82b1-11dd-ad27-0f66e57d2035
Parts:
- added R23: 100k, symbol R_MINI
Connections:
- net labels added: AVDD1, AVSS1
- wire segments 253 -> 256
Other:
- note added: "3M 950450-7203 mates with 3M 951250-7"
- note added: "ADS1298 Notes:\n - capacitors are X7R, 6.3V, 10% or better\n - pull-up resistors can be standard 5%\n - connectors for precision off-board signals (CLK, WCT) should be\n RF coaxial connectors such as Hirose U.FL or Tyco UMCC\n - ADM811 will de-assert RESET 140ms+ after 3.3V is valid\n to give time for other regulators to stabilize\n - AGND and DGND should be separate layers in the PCB stack-up"
- note added: "AVDD"
- note added: "AVSS"
- note added: "CLKSEL=0 for External Clock\nCLKSEL=1 for Internal Clock\nas per datasheet Pg24"
- note added: "DVDD"
- note added: "ERC Fixes"
- note added: "GALVANIC ISOLATION"
- note added: "Notes:\n - ADuM_401 chosen for medical-grade isolation - 5kVDC\n - ADuM4401 only needs to be populated in multi-ADS1298 systems\n - require 4-layer board to proper isolator layout per Analog AppNote AN-0971\n - series resistors should be 1% or better"
- note added: "Notes:\n - resistors should be 0.1%, 50ppm or better\n - Panasonic ERA-6A are 0805, +/-25ppm, 0.1%, 0.20USD\n - Susumu RG are 0805, +/-10ppm, 0.05%, 1.00USD\n - capacitors are X7R, 6.3V, 10% or better"
- note added: "Power Supply Notes:\n - all components chosen for low noise, high PSRR, and RF compatibility\n - capacitors are X5R, 6.3V, 20% or better\n - additional supply filtering on recommendation of TI AppNote SPRAB36A Pg29"
- note added: "REFERENCE"
- note added: "RESET Supervisor"
- note added: "Tie START low to control\nconversions via commands.\nAs per datasheet Pg34"
- moved on the sheet: C2, C34, C35, C36, C41, C42, C43, C44, C46, C47, C48, F1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
