File: ADS1298/ADS1298.sch (KiCad schematic (older format))
At the start: 269 parts, among them IC1 ADS1298, IC2 ADuM6401, IC3 ADuM4401, IC4 ADM811, IC5 REF5025, IC6 OPA211, P1 ADS_Sensors, P2 PCB_BoardCut, U1 ADS1298_Control, U2 TPS79230, U3 TPS79101, U4 TPS60403, U5 TPS72325

Commit message: Minor update to ADS1298 project.
git-svn-id: http://opendous.googlecode.com/svn/trunk/Current_Designs@189 3806c4c6-82b1-11dd-ad27-0f66e57d2035
Other:
- note added: "Consider Hirose FX15S-51S-0.5SH Receptacle and FX15S-51P-C\nPlug which are shielded RA SMT Connectors each about 3USD"
Changed lines of the file:
@@
-EESchema Schematic File Version 2  date 17/04/2010 17:11:51
+EESchema Schematic File Version 2  date 18/04/2010 02:44:13
 LIBS:opendous
 LIBS:device
@@
 Sheet 1 1
 Title "ADS1298 Base Board"
-Date "17 apr 2010"
+Date "18 apr 2010"
 Rev "1.0"
 Comp "Opendous Inc. (www.opendous.org)"
@@
 Comment4 "http://www.opendous.org/BioSensorPlatform"
 $EndDescr
+Text Notes 8050 6450 0    60   ~ 0
+Consider Hirose FX15S-51S-0.5SH Receptacle and FX15S-51P-C\nPlug which are shielded RA SMT Connectors each about 3USD
 Text Notes 1950 1650 0    30   ~ 0
 GND Fence surrounds\ncircuit to limit EMI
@@
 	0    1    1    0
 $EndComp
-Text Notes 8400 6250 0    60   ~ 0
+Text Notes 8400 6200 0    60   ~ 0
 Sullins FFMD-25-D Cable for Female Headers 20USD
-Text Notes 8400 6350 0    60   ~ 0
+Text Notes 8400 6300 0    60   ~ 0
 Sullins FFSD-25-D Cable for Male Headers 20USD
-Text Notes 8100 6050 0    60   ~ 0
+Text Notes 8100 6000 0    60   ~ 0
 Use Sullins SFH31-NPPB-D25-SP-BK (Female Header) 3USD
 Text Label 2000 6250 0    20   ~ 0
@@
 Text Notes 5450 550  0    40   ~ 0
 CLKSEL=0 for External Clock\nCLKSEL=1 for Internal Clock\nas per datasheet Pg24
-Text Notes 8100 6150 0    60   ~ 0
+Text Notes 8100 6100 0    60   ~ 0
 Mates with Sullins SBH31-NBPB-D25-ST-BK (Male Header) 3USD
 Text Notes 1850 2850 0    40   ~ 0
@@
 Text Notes 3500 3400 0    60   ~ 0
 DVDD
-Text Notes 8650 5850 0    60   ~ 0
+Text Notes 8650 5800 0    60   ~ 0
 1.27mm*1.27mm Dual Row 25x2 Header
 $Comp

Commit message: Corrected schematic and layout negative voltage regulator pinout.  Updated KiCAD libraries.
git-svn-id: http://opendous.googlecode.com/svn/trunk/Current_Designs@193 3806c4c6-82b1-11dd-ad27-0f66e57d2035
Parts:
- removed IC2: ADuM6401, symbol ADUMX401
- removed U5: TPS72325, symbol TPS736XX
- added IC2: ADuM6401, symbol ADUM6401
- added U5: TPS72325, symbol TPS723XX
- U3: value TPS79101 -> TPS79201
Connections:
- wire segments 376 -> 379
- no-connect marks 10 -> 14
Other:
- note added: "Note: Install R20, R21 if using TPS72301 or LT1964; select resistors appropriately"
- note added: "TPS72301, LT1964"
- note removed: "Note: Install R20, R21 if using TPS72301"
- note removed: "TPS72301"
- note removed: "TPS79201"
- moved on the sheet: L19

Commit message: Updated design files which now pass all ERC tests.
git-svn-id: http://opendous.googlecode.com/svn/trunk/Current_Designs@197 3806c4c6-82b1-11dd-ad27-0f66e57d2035
Other:
- note added: "Notes:\n - do not populate L18 FB if using external reference\n - resistors should be 0.1%, 50ppm or better\n - use 0.1% resistors with the 0.1% version of the REF5025\n and 0.05% resistors with the 0.05% version\n - Panasonic ERA-6A are 0805, +/-25ppm, 0.1%, 0.20USD\n - Susumu RG are 0805, +/-10ppm, 0.05%, 1.00USD\n - capacitors are X5R, 6.3V, 10% or better unless noted\n - 1206 capacitors are t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"
- note removed: "Notes:\n - do not populate L18 FB if using external reference\n - resistors should be 0.1%, 50ppm or better\n - Panasonic ERA-6A are 0805, +/-25ppm, 0.1%, 0.20USD\n - Susumu RG are 0805, +/-10ppm, 0.05%, 1.00USD\n - capacitors are X5R, 6.3V, 10% or better unless noted\n - 1206 capacitors are tantalum 6.3V with <300mOhm ESR"
Changed lines of the file:
@@
-EESchema Schematic File Version 2  date 01/05/2010 13:30:25
+EESchema Schematic File Version 2  date 09/05/2010 02:06:27
 LIBS:opendous
 LIBS:device
@@
 LIBS:valves
 LIBS:power
+LIBS:ADS1298-cache
 EELAYER 24  0
 EELAYER END
@@
 Sheet 1 1
 Title "ADS1298 Base Board"
-Date "1 may 2010"
+Date "9 may 2010"
 Rev "1.0"
 Comp "Opendous Inc. (www.opendous.org)"
@@
 AVDD1
 Text Notes 5450 4800 0    50   ~ 0
-Design Notes:\n - capacitors are X7R, 6.3V, 20% or better unless otherwise noted\n - pull-up resistors can be standard 5%\n - connectors for precision off-board signals (CLK, RLDINV) should be RF\n    coaxial connectors such as Tyco UMCC or Hirose U.FL (which are footprint compatible)\n - ADM811 will de-assert RESET 140ms+ after 3.3V is valid\n    to give time for other regulators to stabilize\n - AGND and DGND should be separate layers in the PCB stack-up\n - power vias should be 20mil or larger to lower impedance\n - place power and isolation components on bottom of PCB and analog\n    circuitry on top\n - VREF and VCAP1 caps C11, C17 should be highest quality possible\n - Staggered AGND on sensor connector is for differential pair isolation
+Design Notes:\n - capacitors are X7R, 6.3V, 20% or better unless otherwise noted\n - pull-up resistors can be standard 5%\n - connectors for precision off-board signals (CLK, RLDINV) should be RF\n    coaxial connectors such as Tyco UMCC or Hirose U.FL (which are footprint compatible)\n - ADM811 will de-assert RESET 140ms+ after 3.3V is valid\n    to give time for other regulators to stabilize\n - AGND and DGND should be separate layers in the PCB stack-up\n - power vias should be 20mil or larger to lower impedance\n - place power and isolation components on bottom of PCB and analog\n    circuitry on top\n - VREF and VCAP1 caps C11, C17 should be highest quality possible\n - Staggered AGND on ADS_Sensors connector is for differential pair isolation
 Text Notes 5350 2200 0    40   ~ 0
 Tie START low to control\nconversions via commands,\nAs per datasheet Pg34
@@
 RESET Supervisor
 Text Notes 3400 6400 0    40   ~ 0
-Notes:\n - do not populate L18 FB if using external reference\n - resistors should be 0.1%, 50ppm or better\n - Panasonic ERA-6A are 0805, +/-25ppm, 0.1%, 0.20USD\n - Susumu RG are 0805, +/-10ppm, 0.05%, 1.00USD\n - capacitors are X5R, 6.3V, 10% or better unless noted\n - 1206 capacitors are tantalum 6.3V with <300mOhm ESR
+Notes:\n - do not populate L18 FB if using external reference\n - resistors should be 0.1%, 50ppm or better\n - use 0.1% resistors with the 0.1% version of the REF5025\n    and 0.05% resistors with the 0.05% version\n - Panasonic ERA-6A are 0805, +/-25ppm, 0.1%, 0.20USD\n - Susumu RG are 0805, +/-10ppm, 0.05%, 1.00USD\n - capacitors are X5R, 6.3V, 10% or better unless noted\n - 1206 capacitors are tantalum 6.3V with <300mOhm ESR
 Text Notes 3350 6300 0    60   ~ 0
 External REFERENCE
