File: ADS1298/ADS1298_2Layer_Test/ADS1298_2Layer_Test.sch (KiCad schematic (older format))
At the start: 269 parts, among them IC1 ADS1298, IC2 ADuM6401, IC3 ADuM4401, IC4 ADM811, IC5 REF5025, IC6 OPA211, P1 ADS_Sensors, P2 PCB_BoardCut, U1 ADS1298_Control, U2 TPS79230, U3 TPS79101, U4 TPS60403, U5 TPS72325

Commit message: Updated ADS1298 project.  Test 2-layer board is now complete.
git-svn-id: http://opendous.googlecode.com/svn/trunk/Current_Designs@185 3806c4c6-82b1-11dd-ad27-0f66e57d2035
Parts:
- removed C41: 10p, symbol C_MINI
- removed C42, C44: 0u1, symbol C_MINI
- removed C43: 10u, symbol C_MINI
- removed C45, C46: 22uF, symbol C_MINI
- removed C47: 100uF, symbol CP_TANTALUM_MINI
- removed IC5: REF5025, symbol REF50XX
- removed IC6: OPA211, symbol OPA211
- removed L18: FB, symbol L_MINI
- removed R10, R12: 47k, symbol R_MINI
- removed R22: 100k, symbol R_MINI
- removed R23, R24: 100, symbol R_MINI
- removed R25: 0, symbol R_MINI
- removed TP2: RF-TP, symbol RF-TP
- removed TP4: CONN_1, symbol CONN_1
- added V149, V150, V151, V152, V153, V154, V155, V156, V157, V158, V159, V160, V161, V162, V163, V164, V165, V166, V167, V168: VIA, symbol VIA
Connections:
- net labels removed: GNDFENCE, VREFP
- wire segments 376 -> 384
- no-connect marks 10 -> 14
Other:
- note added: "AVDD is filtered OUT25"
- note added: "Could not route on 2-layers"
- note added: "Only AVDD was available to route nPWDN on 2-layers"
- note added: "START is low to control\nconversions via commands,\nAs per datasheet Pg34"
- note added: "Sullins SBH31-NBPB-D25-ST-BK (Male Header) 3USD"
- note added: "Sullins SFH31-NPPB-D25-SP-BK (Female Header) 3USD"
- note removed: "1206"
- note removed: "DNP if using\nExternal\nReference"
- note removed: "External REFERENCE"
- note removed: "Mates with Sullins SBH31-NBPB-D25-ST-BK (Male Header) 3USD"
- note removed: "Notes:\n - do not populate L18 FB if using external reference\n - resistors should be 0.1%, 50ppm or better\n - Panasonic ERA-6A are 0805, +/-25ppm, 0.1%, 0.20USD\n - Susumu RG are 0805, +/-10ppm, 0.05%, 1.00USD\n - capacitors are X5R, 6.3V, 10% or better unless noted\n - 1206 capacitors are tantalum 6.3V with <300mOhm ESR"
- note removed: "Tie START low to control\nconversions via commands,\nAs per datasheet Pg34"
- note removed: "Use Sullins SFH31-NPPB-D25-SP-BK (Female Header) 3USD"
- moved on the sheet: C11, P1, V105, V107, V108, V109, V110, V111, V112, V113, V114, V115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

Commit message: Corrected schematic and layout negative voltage regulator pinout.  Updated KiCAD libraries.
git-svn-id: http://opendous.googlecode.com/svn/trunk/Current_Designs@193 3806c4c6-82b1-11dd-ad27-0f66e57d2035
Parts:
- removed U5: TPS72325, symbol TPS736XX
- added U5: TPS72325, symbol TPS723XX
- U3: value TPS79101 -> TPS79201
Other:
- note added: "Note: Install R20, R21 if using TPS72301 or LT1964; select resistors appropriately"
- note added: "REWORK NOTE: In Revision 1.0 TPS79101 was used for U3 (TPS79201)\nbut has an active-low EN pin so connect appropriately or use the TPS79201"
- note added: "REWORK NOTE: In Revision 1.0 pins IN\nand GND of TPS72325 (U5) were reversed\nCurrent Revision of Board Layout is correct"
- note added: "TPS72301, LT1964"
- note removed: "Note: Install R20, R21 if using TPS72301"
- note removed: "TPS72301"
- note removed: "TPS79201"
Changed lines of the file:
@@
-EESchema Schematic File Version 2  date 17/04/2010 17:11:15
+EESchema Schematic File Version 2  date 01/05/2010 13:29:16
 LIBS:opendous
 LIBS:device
@@
 LIBS:valves
 LIBS:power
-LIBS:ADS1298_2Layer_Test-cache
 EELAYER 24  0
 EELAYER END
@@
 Sheet 1 1
 Title "ADS1298 Base Board 2-Layer Test"
-Date "17 apr 2010"
-Rev "1.0"
+Date "1 may 2010"
+Rev "1.1"
 Comp "Opendous Inc. (www.opendous.org)"
 Comment1 "http://creativecommons.org/licenses/by/3.0/"
@@
 Comment4 "http://www.opendous.org/BioSensorPlatform"
 $EndDescr
-Text Label 6650 8150 2    20   ~ 0
-GPIO2-RESP_BLK
-NoConn ~ 10500 5100
-NoConn ~ 9700 5100
-NoConn ~ 9700 5200
+$Comp
+L GND #PWR01
+U 1 1 4BDC5F0F
+P 6000 8150
+F 0 "#PWR01" H 6000 8150 30  0001 C CNN
+F 1 "GND" H 6000 8080 30  0001 C CNN
+	1    6000 8150
+	1    0    0    -1
+$EndComp
+Text Notes 3350 6500 0    60   ~ 0
+REWORK NOTE: In Revision 1.0 TPS79101 was used for U3 (TPS79201)\nbut has an active-low EN pin so connect appropriately or use the TPS79201
+Connection ~ 1050 4650
+Wire Wire Line
+	1050 5050 1050 4650
 Connection ~ 10750 4600
 Wire Wire Line
@@
 Connection ~ 10750 4400
 Wire Wire Line
-	10500 4400 10750 4400
+	10750 4400 10500 4400
 Wire Wire Line
 	9450 3100 9450 4500
@@
 Connection ~ 1850 7450
 Wire Wire Line
-	1850 7450 1850 7350
+	1850 7350 1850 7450
 Wire Wire Line
 	1700 7150 1700 7050
@@
 	1850 4650 2450 4650
 Wire Wire Line
-	2150 5250 2150 5300
-Wire Wire Line
-	1050 5050 1050 4650
+	2150 5300 2150 5250
 Wire Wire Line
 	900  6850 900  7050
@@
 	900  5400 850  5400
 Connection ~ 900  6850
-Connection ~ 1050 4650
 Wire Wire Line
 	1950 5250 1950 5300
@@
 Connection ~ 2250 7450
 Wire Wire Line
-	2250 7550 2250 7050
-Wire Wire Line
 	1900 700  2400 700
 Connection ~ 2050 700
@@
 Wire Wire Line
 	6550 7900 6550 7950
+Wire Wire Line
+	2250 7050 2250 7500
+$Comp
+L TPS79101 U3
+U 1 1 4BB6CABB
+P 1450 4850
+F 0 "U3" H 1650 4550 40  0000 C CNN
+F 1 "TPS79201" H 1450 5150 45  0000 C CNN
+	1    1450 4850
+	1    0    0    -1
+$EndComp
+Text Notes 3350 7050 0    60   ~ 0
+REWORK NOTE: In Revision 1.0 pins IN\nand GND of TPS72325 (U5) were reversed\nCurrent Revision of Board Layout is correct
+$Comp
+L TPS723XX U5
+U 1 1 4BDC3FFE
+P 1300 6950
+F 0 "U5" H 1500 6700 40  0000 C CNN
+F 1 "TPS72325" H 1300 7150 45  0000 C CNN
+	1    1300 6950
+	1    0    0    -1
+$EndComp
+Text Label 6650 8150 2    20   ~ 0
+GPIO2-RESP_BLK
+NoConn ~ 10500 5100
+NoConn ~ 9700 5100
+NoConn ~ 9700 5200
 NoConn ~ 10500 5200
 $Comp
@@
 $EndComp
 $Comp
-L AGND #PWR01
-U 1 1 4BC93B19
-P 6000 8150
-F 0 "#PWR01" H 6000 8150 40  0001 C CNN
-F 1 "AGND" H 6000 8080 50  0000 C CNN
-	1    6000 8150
-	1    0    0    -1
-$EndComp
-$Comp
 L GND #PWR02
 U 1 1 4BC9356B
@@
 DOUT
 Text Notes 550  7700 0    40   ~ 0
-Note: Install R20, R21 if using TPS72301
+Note: Install R20, R21 if using TPS72301 or LT1964; select resistors appropriately
 Text Notes 1950 7275 0    30   ~ 0
 Optional
 Text Notes 1950 6975 0    30   ~ 0
 Optional
-Text Notes 1150 6700 0    40   ~ 0
-TPS72301
+Text Notes 1025 6700 0    40   ~ 0
+TPS72301, LT1964
 $Comp
 L R_MINI R21
@@
 	-1   0    0    1
 $EndComp
-Text Notes 1300 4500 0    40   ~ 0
-TPS79201
 Text Notes 1800 3400 0    40   ~ 0
 TPS79133
@@
 L AGND #PWR0117
 U 1 1 4BB6CDB5
-P 2250 7550
-F 0 "#PWR0117" H 2250 7550 40  0001 C CNN
-F 1 "AGND" H 2250 7480 50  0000 C CNN
-	1    2250 7550
+P 2250 7500
+F 0 "#PWR0117" H 2250 7500 40  0001 C CNN
+F 1 "AGND" H 2250 7430 50  0000 C CNN
+	1    2250 7500
 	1    0    0    -1
 $EndComp
@@
 	0    1    1    0
 $EndComp
-$Comp
-L TPS736XX U5
-U 1 1 4BB6CAF0
-P 1300 6950
-F 0 "U5" H 1500 6700 40  0000 C CNN
-F 1 "TPS72325" H 1300 7150 45  0000 C CNN
-	1    1300 6950
-	1    0    0    -1
-$EndComp
-$Comp
-L TPS79101 U3
-U 1 1 4BB6CABB
-P 1450 4850
-F 0 "U3" H 1650 4550 40  0000 C CNN
-F 1 "TPS79101" H 1450 5150 45  0000 C CNN
-	1    1450 4850
-	1    0    0    -1
-$EndComp
 NoConn ~ 8300 3900

Commit message: Updated design files which now pass all ERC tests.
git-svn-id: http://opendous.googlecode.com/svn/trunk/Current_Designs@197 3806c4c6-82b1-11dd-ad27-0f66e57d2035
Parts:
- removed IC2: ADuM6401, symbol ADUMX401
- added IC2: ADuM6401, symbol ADUM6401
Connections:
- net labels added: GNDFENCE
- wire segments 384 -> 387
- no-connect marks 14 -> 16
Other:
- moved on the sheet: L19
