File: BioSensorPlatform/BioSensorPlatform.sch (KiCad schematic (older format))
At the start: 287 parts, among them IC1 ADS1298, P1 GPIO, P2 Interface, P3 AN, U2 79230, U3 79201, U4 60403, U5 72325

Commit message: Updated designs with latest Gerber archives.  Added MultiAdaptor_v2 design which now includes SC70-8 and SOT23-8 footprints.  Also added AudioOpAmpTester design which is a simple stereo audio amplifier with a +/- 15V boost converter power supply that runs off a 9V battery.
git-svn-id: http://opendous.googlecode.com/svn/trunk/Current_Designs@262 3806c4c6-82b1-11dd-ad27-0f66e57d2035
Parts:
- added C10: 1n5, symbol C_MINI
- added R4: 1M, symbol R_MINI
Connections:
- wire segments 391 -> 392
