File: LT1945/LT1945.sch (KiCad schematic (older format))
At the start: 30 parts, among them IC91 LT1945, P91 VIN, P92 VOUT

Commit message: Updated designs with latest Gerber archives.  Added MultiAdaptor_v2 design which now includes SC70-8 and SOT23-8 footprints.  Also added AudioOpAmpTester design which is a simple stereo audio amplifier with a +/- 15V boost converter power supply that runs off a 9V battery.
git-svn-id: http://opendous.googlecode.com/svn/trunk/Current_Designs@262 3806c4c6-82b1-11dd-ad27-0f66e57d2035
Parts:
- added BT1: BATTERY, symbol BATTERY
- added C97: 10u, symbol C_MINI
- added D94: NEG_ON, symbol D_LED
- added D95: POS_ON, symbol D_LED
- added P1: 9V, symbol CONN_2
- added R83, R93: 2k, symbol R_MINI
- added V912, V913, V914: VIA, symbol VIA
- D91, D92, D93: value MBR120 -> MBR140
- R82: value R_MINI -> 24k9
- R92: value R_MINI -> 100k
Connections:
- net labels added: FB2, SW2, nFB1, nSHDN1, nSHDN2
- wire segments 38 -> 57
Other:
- note added: "+"
- note added: "-"
- note added: "Note: Depending on output voltage, can use any\nSOD-123 Schottky rated 0.4A+ instead of MBR140"
- note added: "Note: R82 and R92 can also be changed to use\nstandard resistors that get the output voltage\ncloser to your intended output voltage."
- note added: "Note: The 10uH 7045-size inductors have been\nchosen for high output current when using a 1.5V\nbattery to generate +/- (2V to 5V). Refer to the\nLT1945 datasheet for component selection calculations."
- note added: "R81 = ((|VSUP1| - 1.23) / ((1.23 / 24900) + (0.000002)))"
- note added: "R91 = 100000((VSUP2 / 1.23) - 1)"
- moved on the sheet: P91, P92, V900, V901, V902, V903, V904, V905, V906, V907, V908, V909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
