File: AudioOpAmpTester/Audio_OpAmp_Tester.sch (KiCad schematic (older format))
At the start: 208 parts, among them IC1 OpAmp, IC2 OpAmp, IC91 LT1945, IC92 TPS7A3001, IC93 TPS7A4901, P1 9V, P2 8DIP, P3 8SOIC, P4 8DIP, P5 8MSOP, P91 VIN, P92 VOUT, U1 IN, U2 OUT

Commit message: Updated Audio OpAmp Tester design.
git-svn-id: http://opendous.googlecode.com/svn/trunk/Current_Designs@265 3806c4c6-82b1-11dd-ad27-0f66e57d2035
Parts:
- added Mask1, Mask2, Mask3, Mask4, Mask5, Mask6, Mask7, Mask8: CONN_1, symbol CONN_1
- R10, R8: value 100k -> 1k
- R11, R12: value 0 -> 10
- R7, R9: value 100k -> 10k
Connections:
- no-connect marks 2 -> 10
Other:
- note added: "Amplification equals R7/R8+1 = 10k/1k+1 = 11"
- note added: "Amplification equals R9/R10+1 = 10k/1k+1 = 11"
- note added: "Gain of 11 = 20.9dB\nFor audio frequencies the root Hz is sqrt(20000-20) = 141.35\nIf using the OPA2211 OpAmp with 1.1nV/sqrt(Hz) voltage noise\nthe Equivalent Input Noise is 1.1*141.35 = 155.49 nV\nOutput noise is input noise multiplied by gain:\n155.49 * 11 = 1710 nV\nSignal-to-Noise therefore = 20*log(1V / (1710*(10^-9))) = 20log(584795) = 115dB\nWith a gain of 2 it would be 20log(1/((141.35*1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"
- note added: "These mask cutouts prevent the GND\nguard shield from capacitively coupling\nwith the LT1945 GND."
- note added: "These mask cutouts prevent the GND\nguard shield from capacitively coupling\nwith the analog GND."
- note removed: "Note: The 10uH 7045-size inductors have been\nchosen for high output current when using a 1.5V\nbattery to generate +/- (2V to 5V). Refer to the\nLT1945 datasheet for component selection calculations."
Changed lines of the file:
@@
-EESchema Schematic File Version 2  date 21/03/2011 09:08:14
-LIBS:opendous
+EESchema Schematic File Version 2  date 6/12/2011 3:38:19 PM
 LIBS:device
 LIBS:transistors
@@
 EELAYER END
 $Descr A4 11700 8267
+encoding utf-8
 Sheet 1 1
 Title "Audio OpAmp Tester"
-Date "21 mar 2011"
+Date "12 jun 2011"
 Rev "1.0"
 Comp "Opendous Inc. (www.opendous.org)"
@@
 Comment4 "http://www.opendous.org/AudioOpAmpTester"
 $EndDescr
+$Comp
+L CONN_1 Mask5
+U 1 1 4DF50BEF
+P 6750 2850
+F 0 "Mask5" H 6830 2850 40  0000 L CNN
+F 1 "CONN_1" H 6750 2905 30  0001 C CNN
+	1    6750 2850
+	-1   0    0    1
+$EndComp
+$Comp
+L CONN_1 Mask6
+U 1 1 4DF50BEE
+P 6750 2950
+F 0 "Mask6" H 6830 2950 40  0000 L CNN
+F 1 "CONN_1" H 6750 3005 30  0001 C CNN
+	1    6750 2950
+	-1   0    0    1
+$EndComp
+$Comp
+L CONN_1 Mask8
+U 1 1 4DF50BED
+P 7300 2950
+F 0 "Mask8" H 7380 2950 40  0000 L CNN
+F 1 "CONN_1" H 7300 3005 30  0001 C CNN
+	1    7300 2950
+	1    0    0    1
+$EndComp
+$Comp
+L CONN_1 Mask7
+U 1 1 4DF50BEC
+P 7300 2850
+F 0 "Mask7" H 7380 2850 40  0000 L CNN
+F 1 "CONN_1" H 7300 2905 30  0001 C CNN
+	1    7300 2850
+	1    0    0    1
+$EndComp
+NoConn ~ 6900 2850
+NoConn ~ 7150 2850
+NoConn ~ 7150 2950
+NoConn ~ 6900 2950
+Text Notes 6650 2650 0    30   ~ 0
+These mask cutouts prevent the GND\nguard shield from capacitively coupling\nwith the LT1945 GND.
+Text Notes 5400 2650 0    30   ~ 0
+These mask cutouts prevent the GND\nguard shield from capacitively coupling\nwith the analog GND.
+NoConn ~ 5650 2950
+NoConn ~ 5900 2950
+NoConn ~ 5900 2850
+NoConn ~ 5650 2850
+$Comp
+L CONN_1 Mask3
+U 1 1 4DF50955
+P 6050 2850
+F 0 "Mask3" H 6130 2850 40  0000 L CNN
+F 1 "CONN_1" H 6050 2905 30  0001 C CNN
+	1    6050 2850
+	1    0    0    1
+$EndComp
+$Comp
+L CONN_1 Mask4
+U 1 1 4DF50954
+P 6050 2950
+F 0 "Mask4" H 6130 2950 40  0000 L CNN
+F 1 "CONN_1" H 6050 3005 30  0001 C CNN
+	1    6050 2950
+	1    0    0    1
+$EndComp
+$Comp
+L CONN_1 Mask2
+U 1 1 4DF5094F
+P 5500 2950
+F 0 "Mask2" H 5580 2950 40  0000 L CNN
+F 1 "CONN_1" H 5500 3005 30  0001 C CNN
+	1    5500 2950
+	-1   0    0    1
+$EndComp
+$Comp
+L CONN_1 Mask1
+U 1 1 4DF50941
+P 5500 2850
+F 0 "Mask1" H 5580 2850 40  0000 L CNN
+F 1 "CONN_1" H 5500 2905 30  0001 C CNN
+	1    5500 2850
+	-1   0    0    1
+$EndComp
+Text Notes 950  5900 0    60   ~ 0
+Gain of 11 = 20.9dB\nFor audio frequencies the root Hz is sqrt(20000-20) = 141.35\nIf using the OPA2211 OpAmp with 1.1nV/sqrt(Hz) voltage noise\nthe Equivalent Input Noise is 1.1*141.35 = 155.49 nV\nOutput noise is input noise multiplied by gain:\n155.49 * 11 = 1710 nV\nSignal-to-Noise therefore = 20*log(1V / (1710*(10^-9))) = 20log(584795) = 115dB\nWith a gain of 2 it would be 20log(1/((141.35*1.1*2)*10^(-9))) = 130dB
+Text Notes 6950 4050 0    60   ~ 0
+Amplification equals R7/R8+1 = 10k/1k+1 = 11
+Text Notes 6950 5950 0    60   ~ 0
+Amplification equals R9/R10+1 = 10k/1k+1 = 11
 Text Label 1500 3550 2    20   ~ 0
 Thermal
@@
 	700  7050 700  7500
 Wire Wire Line
-	600  7150 600  7200
-Wire Wire Line
-	700  7150 600  7150
+	600  7200 600  7150
+Wire Wire Line
+	600  7150 700  7150
 Connection ~ 700  7500
 Connection ~ 700  7450
@@
 	3450 7500 3450 7150
 Wire Wire Line
-	3650 7150 3650 7200
-Wire Wire Line
-	3750 7150 3650 7150
+	3650 7200 3650 7150
+Wire Wire Line
+	3650 7150 3750 7150
 Wire Wire Line
 	3450 7150 3350 7150
 Wire Wire Line
-	3750 7500 3750 7150
+	3750 7150 3750 7500
 Connection ~ 3450 7500
 Connection ~ 3450 7450
@@
 	5500 5250 5500 5250
 Wire Wire Line
-	5500 5700 5500 5250
-Wire Wire Line
-	6300 5700 5500 5700
+	5500 5250 5500 5700
+Wire Wire Line
+	5500 5700 6300 5700
 Wire Wire Line
 	6300 6000 6300 6050
@@
 	6300 4500 6300 4550
 Wire Wire Line
-	5500 4200 6300 4200
-Wire Wire Line
-	5500 3750 5500 4200
+	6300 4200 5500 4200
+Wire Wire Line
+	5500 4200 5500 3750
 Wire Wire Line
 	5200 3850 5200 3900
@@
 Connection ~ 10850 2150
 Wire Wire Line
-	10950 2150 10950 2100
-Wire Wire Line
-	10150 2150 10950 2150
+	10950 2100 10950 2150
+Wire Wire Line
+	10950 2150 10150 2150
 Connection ~ 10850 850
 Wire Wire Line
@@
 	9250 2650 9250 2600
 Wire Wire Line
-	9350 2150 9350 2250
+	9350 2250 9350 2150
 Wire Wire Line
 	9350 2400 9250 2400
@@
 Connection ~ 9250 2600
 Wire Wire Line
-	8950 2150 8950 2100
-Wire Wire Line
-	9350 2150 8950 2150
+	8950 2100 8950 2150
+Wire Wire Line
+	8950 2150 9350 2150
 Connection ~ 9050 2150
 Connection ~ 9050 850
@@
 	9350 1300 9250 1300
 Wire Wire Line
-	10450 1050 10450 1100
+	10450 1100 10450 1050
 Connection ~ 10450 850
 Wire Wire Line
@@
 Connection ~ 1850 1050
 Wire Wire Line
-	1750 1050 1750 1000
+	1750 1000 1750 1050
 Wire Wire Line
 	800  1600 800  1650
@@
 Connection ~ 2250 1250
 Wire Wire Line
-	2250 1050 2250 1400
-Wire Wire Line
-	1750 1050 2250 1050
+	2250 1400 2250 1050
+Wire Wire Line
+	2250 1050 1750 1050
 Wire Wire Line
 	3300 1050 3400 1050
@@
 	3150 1400 3150 1500
 Wire Wire Line
-	3650 1500 3150 1500
+	3150 1500 3650 1500
 Wire Wire Line
 	3650 1500 3650 1400
@@
 	10750 1350 10750 1050
 Wire Wire Line
-	10150 1050 10450 1050
+	10450 1050 10150 1050
 Connection ~ 10250 1050
 Wire Wire Line
@@
 	4550 7150 4550 7200
 Wire Wire Line
-	4950 7150 4850 7150
+	4850 7150 4950 7150
 Wire Wire Line
 	4850 7150 4850 7200
@@
 	3000 7150 3000 7200
 Wire Wire Line
-	4950 7500 4950 7150
+	4950 7150 4950 7500
 Wire Wire Line
 	5500 1050 5600 1050
@@
 	9050 1050 9050 1350
 Wire Wire Line
-	5300 1200 5950 1200
-Wire Wire Line
-	5300 1050 5300 1200
-Wire Wire Line
-	4300 1050 5300 1050
+	5950 1200 5300 1200
+Wire Wire Line
+	5300 1200 5300 1050
+Wire Wire Line
+	5300 1050 4300 1050
 Connection ~ 10650 850
 Connection ~ 10650 2150
@@
 	3350 7150 3350 7200
 Wire Wire Line
-	2650 7150 2650 7200
-Wire Wire Line
-	2300 7150 2300 7200
-Wire Wire Line
-	2400 7150 2300 7150
-Wire Wire Line
-	2400 7500 2400 7150
+	2650 7200 2650 7150
+Wire Wire Line
+	2300 7200 2300 7150
+Wire Wire Line
+	2300 7150 2400 7150
+Wire Wire Line
+	2400 7150 2400 7500
 Connection ~ 2400 7500
 Connection ~ 2400 7450
@@
 Connection ~ 2750 7500
 Wire Wire Line
-	2750 7150 2650 7150
-Wire Wire Line
-	2750 7500 2750 7150
+	2650 7150 2750 7150
+Wire Wire Line
+	2750 7150 2750 7500
 Wire Wire Line
 	10400 4150 10400 4200
@@
 	1900 7150 1900 7200
 Wire Wire Line
-	1200 7150 1200 7200
-Wire Wire Line
-	1300 7150 1200 7150
-Wire Wire Line
-	1300 7500 1300 7150
+	1200 7200 1200 7150
+Wire Wire Line
+	1200 7150 1300 7150
+Wire Wire Line
+	1300 7150 1300 7500
 Connection ~ 1300 7500
 Connection ~ 1300 7450
@@
 P 5850 3700
 F 0 "IC2" H 5650 3300 50  0000 C CNN
-F 1 "OpAmp" H 5550 4000 35  0000 C CNN
+F 1 "OpAmp" H 5650 4000 35  0000 C CNN
 	1    5850 3700
 	1    0    0    -1
@@
 P 6300 5900
 F 0 "R10" V 6275 5950 25  0000 C CNN
-F 1 "100k" V 6325 5950 20  0000 C CNN
+F 1 "1k" V 6325 5950 20  0000 C CNN
 	1    6300 5900
 	0    1    1    0
@@
 P 6300 5500
 F 0 "R9" V 6275 5550 25  0000 C CNN
-F 1 "100k" V 6325 5550 20  0000 C CNN
+F 1 "10k" V 6325 5550 20  0000 C CNN
 	1    6300 5500
 	0    1    1    0
@@
 P 6550 5200
 F 0 "R12" H 6480 5250 25  0000 C CNN
-F 1 "0" H 6620 5250 20  0000 C CNN
+F 1 "10" H 6620 5250 20  0000 C CNN
 	1    6550 5200
 	1    0    0    -1
@@
 P 6550 3700
 F 0 "R11" H 6480 3750 25  0000 C CNN
-F 1 "0" H 6620 3750 20  0000 C CNN
+F 1 "10" H 6620 3750 20  0000 C CNN
 	1    6550 3700
 	1    0    0    -1
@@
 P 6300 4000
 F 0 "R7" V 6275 4050 25  0000 C CNN
-F 1 "100k" V 6325 4050 20  0000 C CNN
+F 1 "10k" V 6325 4050 20  0000 C CNN
 	1    6300 4000
 	0    1    1    0
@@
 P 6300 4400
 F 0 "R8" V 6275 4450 25  0000 C CNN
-F 1 "100k" V 6325 4450 20  0000 C CNN
+F 1 "1k" V 6325 4450 20  0000 C CNN
 	1    6300 4400
 	0    1    1    0
@@
 	1    0    0    -1
 $EndComp
-Text Notes 10900 975  0    25   ~ 0
+Text Notes 10710 975  0    25   ~ 0
 25V+
-Text Notes 10900 2275 0    25   ~ 0
+Text Notes 10710 2275 0    25   ~ 0
 25V+
 $Comp
@@
 	1    0    0    -1
 $EndComp
-Text Notes 6650 1550 0    50   ~ 0
-Note: The 10uH 7045-size inductors have been\nchosen for high output current when using a 1.5V\nbattery to generate +/- (2V to 5V).  Refer to the\nLT1945 datasheet for component selection calculations.
 Text Notes 6650 1300 0    50   ~ 0
 Note: Depending on output voltage, can use any\nSOD-123 Schottky rated 0.4A+ instead of MBR140

Commit message: Updated Bill of Materials for the Audio OpAmp Tester design.
git-svn-id: http://opendous.googlecode.com/svn/trunk/Current_Designs@268 3806c4c6-82b1-11dd-ad27-0f66e57d2035
Parts:
- C11, C14: value 0u1 -> u033
- C12, C13: value 220u -> 100u
- C97: value 10u -> 4u7
- R83, R93: value 2k -> 5k
Changed lines of the file:
@@
-EESchema Schematic File Version 2  date 6/12/2011 3:38:19 PM
+EESchema Schematic File Version 2  date 6/15/2011 10:22:22 AM
 LIBS:device
 LIBS:transistors
@@
 Sheet 1 1
 Title "Audio OpAmp Tester"
-Date "12 jun 2011"
+Date "15 jun 2011"
 Rev "1.0"
 Comp "Opendous Inc. (www.opendous.org)"
@@
 P 10400 4300
 F 0 "C14" V 10350 4350 30  0000 C CNN
-F 1 "0u1" V 10450 4350 25  0000 C CNN
+F 1 "u033" V 10450 4350 25  0000 C CNN
 	1    10400 4300
 	0    1    1    0
@@
 P 10200 4300
 F 0 "C11" V 10150 4350 30  0000 C CNN
-F 1 "0u1" V 10250 4350 25  0000 C CNN
+F 1 "u033" V 10250 4350 25  0000 C CNN
 	1    10200 4300
 	0    1    1    0
@@
 P 10850 2250
 F 0 "C13" V 10800 2350 30  0000 C CNN
-F 1 "220u" V 10900 2350 25  0000 C CNN
+F 1 "100u" V 10900 2350 25  0000 C CNN
 	1    10850 2250
 	0    1    1    0
@@
 P 10850 950
 F 0 "C12" V 10900 850 30  0000 C CNN
-F 1 "220u" V 10800 850 25  0000 C CNN
+F 1 "100u" V 10800 850 25  0000 C CNN
 	1    10850 950
 	0    -1   -1   0
@@
 P 1850 1150
 F 0 "C97" V 1800 1200 30  0000 C CNN
-F 1 "10u" V 1900 1200 25  0000 C CNN
+F 1 "4u7" V 1900 1200 25  0000 C CNN
 	1    1850 1150
 	0    1    1    0
@@
 P 6050 1500
 F 0 "R93" H 5980 1550 25  0000 C CNN
-F 1 "2k" H 6120 1550 20  0000 C CNN
+F 1 "5k" H 6120 1550 20  0000 C CNN
 	1    6050 1500
 	1    0    0    -1
@@
 P 6350 1200
 F 0 "R83" H 6280 1250 25  0000 C CNN
-F 1 "2k" H 6420 1250 20  0000 C CNN
+F 1 "5k" H 6420 1250 20  0000 C CNN
 	1    6350 1200
 	-1   0    0    -1
