File: Opennect-Touchscreen_LCD/Opennect-Touchscreen_LCD.sch (KiCad schematic (older format))
At the start: 144 parts, among them IC1 LOGIC-MUX_2TO1, IC2 EEPROM, IC3 LOGIC-INVERTER, IC4 LVC2T45, IC5 PCA9306, IC6 CAT4237, IC7 LVC2T45, IC8 STMPE610, P1 Breakout, U1 Opennect-Module-MCU_3V3to5V, U2 Opennect-Controller-MCU_3V3to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, U3 COG-C172MVHC-04

Commit message: Updated Opennect Touchscreen-LCD and USB Protocol Analyzer Front-End designs.
git-svn-id: http://opendous.googlecode.com/svn/trunk/Current_Designs@277 3806c4c6-82b1-11dd-ad27-0f66e57d2035
Parts:
- added C12, C13: 1u0, symbol C_MINI
- added C14: u01, symbol C_MINI
- added IC9: REG2V8, symbol REGULATOR_SOT23-5
- added V107, V108, V109, V110, V111, V112, V113, V114, V115: VIA, symbol VIA
Connections:
- net labels added: 2V8
- wire segments 266 -> 286
Other:
- note added: "Compatible SOT23-5 Regulators:\nAP7331-28W\nXC6221?28\nNCP3985SN28T1\nLP2985-28DBV\nTC1185-2.8VCT713"
- note added: "nMS needs INVERTER!"
- moved on the sheet: C7, V83, V89
