File: MultiAdaptor/MultiAdaptor.sch (KiCad schematic (older format))
At the start: 30 parts, among them P1 CONN_14, P10 CONN_1, P11 CONN_1, P12 CONN_1, P13 CONN_1, P14 CONN_1, P15 CONN_1, P16 CONN_1, P2 CONN_14, P3 SOT223, P6 SOT143, P7 CONN_1, P8 CONN_1, P9 CONN_1, U1 SOIC28, U10 MSOP10, U2 SOT23, U3 SOT23, U4 SOT23, U5 SOT23, U6 SSOP28, U7 SC70, U8 SC70, U9 SC70

Commit message: Updated MultiAdaptor project files to Revision 2012-06-02.
git-svn-id: http://opendous.googlecode.com/svn/trunk/Current_Designs@310 3806c4c6-82b1-11dd-ad27-0f66e57d2035
Parts:
- removed U4, U5: SOT23, symbol CONN_3X2_DIL
- removed U7, U8: SC70, symbol CONN_3X2_DIL
- removed V1, V2, V3, V4, V5, V6: VIA, symbol VIA
- added U11: SC70-6, symbol CONN_3X2_DIL
- added U4: SOT23-8, symbol CONN_4X2_DIL
- added U5: SOT23-3, symbol CONN_3
- added U8: SC70-8, symbol CONN_4X2_DIL
- U2, U3: value SOT23 -> SOT23-6
- U9: value SC70 -> SC70-6
Connections:
- net labels removed: GND
- wire segments 12 -> 10
Other:
- moved on the sheet: P10, P11, P12, P13, P14, P15, P16, P7, P8, P9, U10
