File: Upconverter/Upconverter-100MHz-13LO-SMS3926-CX2147.sch (KiCad schematic (older format))
At the start: 213 parts, among them IC1 SMS3926, IC2 125, IC3 TPS, P1 RF, P2 IF, T1 CX2147, T2 CX2147, U1 USB-microB, U2 USB-A-Plug, X1 100MHz

Commit message: Added Filter Testing Results and complete files for the Upconverter-100MHz-13LO-SMS3926-CX2147 design.
git-svn-id: http://opendous.googlecode.com/svn/trunk/Current_Designs@330 3806c4c6-82b1-11dd-ad27-0f66e57d2035
Parts:
- C1, C13: value 1uF -> 4.7uF
- C12: value DNP -> 0.01uF
- C3, C9: value 12pF -> 100pF
- R2: value 95R3 -> DNI
- R3: value 75 -> 5R76
- R4: value 95R3 -> 866
- R5: value 39k2 -> DNI
- R6: value 36k5 -> DNI
Connections:
- net labels added: +3.3V
- net labels removed: +2.5V
Other:
- note added: "79333DBV"
- note removed: "73101DBV"
- note removed: "TPS73201DBV"
