File: Upconverter/Upconverter-100MHz-ADE.sch (KiCad schematic (older format))
At the start: 225 parts, among them IC2 125, IC3 TPS, P1 RF, P2 IF, P3 Pa, P4 Pb, U1 USB-microB, U2 USB-A-Plug, U3 ADE, U4 OPENNECT-CLOCK, X1 100MHz

Commit message: Updated Upconverter project with latest design files.
git-svn-id: http://opendous.googlecode.com/svn/trunk/Current_Designs@319 3806c4c6-82b1-11dd-ad27-0f66e57d2035
Parts:
- removed C6: 0.1uF, 0805, symbol C_MINI
- removed C9: 12pF, 0805, symbol C_MINI
- removed D2: Limiter, SC70-3_SOT-323, symbol D_RECTIFIER_SERIES
- removed IC2: 125, SOT23-5, symbol BUFFER_GATE
- removed L2: FB, 0805, symbol L_MINI
- removed P3: Pa, SMA_EndLaunch, symbol BNC
- removed P4: Pb, SMA_EndLaunch, symbol BNC
- removed R1: DNP, 0805, symbol R_MINI
- removed R10: DNI, 0805_Opendous_Labeled, symbol R_MINI
- removed U4: OPENNECT-CLOCK, Opennect_SATA_Molex_67490-1220, symbol OPENNECT-CLOCK
- added C1, C24, C26: 4.7uF, 0805, symbol C_MINI
- added C10: 20pF, 0805, symbol C_MINI
- added C11: 68pF, 0805, symbol C_MINI
- added C21: 56pF, 0805, symbol C_MINI
- added C22: 6.8pF, 0805, symbol C_MINI
- added C23: 330pF, 0805, symbol C_MINI
- added C25: 15pF, 0805, symbol C_MINI
- added C27, C29, C30, C34, C35, C37, C38, C39, C41, C42, C45: 0.1uF, 0805, symbol C_MINI
- added C28, C32: 1000pF, 0805, symbol C_MINI
- added C33, C36, C40, C43, C44, C46: 100pF, 0805, symbol C_MINI
- added D2: MBR120, SOD123, symbol D_SCHOTTKY_SMALL
- added D4: ZENER, SMA_DO214A_Diode, symbol D_ZENER
- added D5: POWERED, 0805, symbol D_LED
- added IC2, IC4: AMP, SOT89-3, symbol AMP_RF_SOT-89
- added IC3: SC4503, SOT23-5, symbol BOOST_DC-DC_SOT23-5
- added IC5: 04, SOT23-6, symbol 74LVC2GU04
- added IC6: RFS1, SOT23-6, symbol RF_SWITCH_SPDT
- added IC7: RFS2, SOT23-6, symbol RF_SWITCH_SPDT
- added IC8: 126, symbol BUFFER_GATE_NONINV
- added JP1: NoiseSource_EN, SIL-2, symbol JUMPER-2-NON
- added JP2: RF_Path_Select, MTS-1x2-C3, symbol JUMPER-3-WITH-GND
- added JP3: OSC_EN, symbol JUMPER-3
- added L13: 6.8nH, 0805, symbol L_MINI
- added L14: 4.7uH, 1206, symbol L_MINI
- added L15, L16: 100nH, 0805, symbol L_MINI
- added L4: 120nH, 0805, symbol L_MINI
- added P1: RF, SMA_EndLaunch, symbol BNC
- added R10: 5k, TrimPOT_TH, symbol TRIMPOT
- added R11: 2k5, 0805, symbol R_MINI
- added R12: 1, 1206, symbol R_MINI
- added R13, R15: DNI, 0603, symbol R_MINI
- added R14: 1k, 0805, symbol R_MINI
- added V169, V170, V171, V172, V173, V174, V175, V176, V177, V178, V179, V180, V181, V182, V183, V184, V185, V186, V187, V188, V189, V190, V191, V192, V193, V194, V195, V196, V197, V198, V199, V200, V201, V202, V203, V204, V205, V206, V207, V208, V209, V210, V211, V212, V213, V214, V215, V216, V217, V218, V219, V220, V221, V222, V223, V224, V225, V226, V227, V228, V229, V230, V231, V232, V233, V234, V235, V236, V237, V238, V239, V240, V241, V242, V243, V244, V245, V246, V247, V248, V249, V250, V251, V252, V253, V254, V255, V256, V257, V258, V259, V260, V261, V262, V263, V264, V265, V266, V267, V268, V269, V270, V271, V272, V273, V274, V275, V276, V277, V278, V279, V280, V281, V282, V283, V284, V285, V286, V287, V288, V289, V290, V291, V292, V293, V294, V295, V296, V297, V298, V299, V300, V301, V302, V303, V304, V305, V306, V307, V308, V309, V310, V311, V312, V313, V314, V315, V316, V317, V318, V319, V320, V321, V322, V323, V324, V325, V326, V327, V328, V329, V330, V331, V332, V333, V334, V335, V336, V337, V338, V339, V340, V341, V342, V343, V344, V345, V346, V347, V348, V349, V350, V351, V352, V353, V354, V355, V356, V357, V358, V359, V360, V361, V362, V363, V364, V365, V366, V367, V368, V369, V370, V371, V372, V373: VIA, 1Pin_20mil_VIA, symbol VIA
- C12: value DNP -> 0.01uF
- C13: value 1uF -> 4.7uF
- C20: value 18pF -> 20pF
- C3: value 12pF -> 100pF
- C31: renamed from C1; value 1uF -> 4.7uF
- C5: value 12pF -> 6.2pF
- C6: renamed from C7; value 82pF -> 100pF
- C7: renamed from C10; value 36pF -> 30pF
- C9: renamed from C11; value 56pF -> 82pF
- D3: value POWER -> POWERED
- L1: value FB -> 47nH
- L3: renamed from L4; value 82nH -> 110nH
- L5: value FB -> 330nH
- P3: renamed from P1; value RF -> OUT
- R2, R4: value 88R7 -> 432
- R3: value 82 -> 11R5
- R5: value 39k2 -> DNI
- R6: value 36k5 -> DNI
- R8: value DNI -> 432k; footprint 0805_Opendous_Labeled -> 0805
- R9: value 0 -> 49k9; footprint 0805_Opendous_Labeled -> 0805
- U2: value USB-A-Plug -> USB-B; footprint CONN_USB-A_Plug_RA_SMT -> CONN_USB_B
- renumbered IC3 to IC1, L3 to L2
Connections:
- net labels added: +12V, +3.3V, AMP1_IN, AMP1_OUT, AMP2_IN, AMP2_OUT, D_Cathode, OSC_EN, OUT, RFS1, RFS2, RF_Passthrough, VDD_RF
- net labels removed: +2.5V, +5V, DGND, LO_BUF
- wire segments 182 -> 370
Other:
- note added: "12V Power Supply"
- note added: "2dB"
- note added: "74LVC2GU"
- note added: "79333DBV"
- note added: "Amplifiers"
- note added: "Avalanche Noise Generator"
- note added: "Bessel Bandpass Filter"
- note added: "Buffer output is\n3.3Vp-p = 14.35dBm\nAfter Attenuator and Filter\nthe LO Level is about 7dBm\naccounting for component variation\n14.35dBm-2-4.5=7.85dBm"
- note added: "Copper Trace"
- note added: "Elliptic (Cauer) Lowpass Filter"
- note added: "Measured loss of 4.5dB at 100MHz"
- note added: "Noise"
- note added: "R12 must be able\nto dissipate 250mW"
- note added: "RF Noise Source"
- note added: "The PTC Fuse has about\n0.5 Ohm resistance"
- note added: "Use a RF amplifier with a\nhigh Noise Figure such as:\nMMG3H21NT1\nSKY65017-70LF"
- note added: "Zener Diodes above 6V use\nAvalanche Breakdown instead\nof Zener Breakdown. Try:\n BZG05C7V5\n 1SMA5922BT3G\n PTZ7.5B"
- note removed: "73101DBV"
- note removed: "<0.3dB ripple below 46MHz\n<1.5dB ripple below 67MHz\n-3dB cutoff at 69MHz\n>40dB attenuation at >88MHz"
- note removed: "A 74LVC1G125 buffer must be powered\nat 2.5V for it to handle a 100MHz+ signal."
- note removed: "Attenuate LO to +10dB"
- note removed: "Attenuator"
- note removed: "Elliptic Lowpass Filter"
- note removed: "Minimum -1dB outside 102MHz to 168MHz\nMinimum -3dB outside 100MHz to 171MHz\nMinimum -30dB outside 85MHz to 198MHz"
- note removed: "TPS73201DBV"
- note removed: "The buffer gate acts as a saturated amplifier\nto reduce amplitude noise in the LO signal."
- moved on the sheet: C12, C13, C14, C15, C16, C17, C18, C19, C2, C20, C3, C31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

Commit message: Added Filter Testing Results and complete files for the Upconverter-100MHz-13LO-SMS3926-CX2147 design.
git-svn-id: http://opendous.googlecode.com/svn/trunk/Current_Designs@330 3806c4c6-82b1-11dd-ad27-0f66e57d2035
Other:
- note added: "Attenuator"
- note removed: "Buffer output is\n3.3Vp-p = 14.35dBm\nAfter Attenuator and Filter\nthe LO Level is about 7dBm\naccounting for component variation\n14.35dBm-2-4.5=7.85dBm"
- note removed: "Measured loss of 4.5dB at 100MHz"
Changed lines of the file:
@@
-EESchema Schematic File Version 2  date 10/4/2012 9:52:59 PM
+EESchema Schematic File Version 2  date 10/5/2012 9:45:18 PM
 LIBS:power
 LIBS:device
@@
 Sheet 1 1
 Title "Upconverter-100MHz-ADE"
-Date "5 oct 2012"
+Date "6 oct 2012"
 Rev "1.0"
 Comp "Opendous Inc."
@@
 Comment4 "For more information visit www.opendous.org/Upconverter"
 $EndDescr
+Text Notes 8350 1000 0    80   ~ 0
+Attenuator
 Wire Wire Line
 	5850 900  5950 900
@@
 	0    -1   -1   0
 $EndComp
-Text Notes 9550 750  0    80   ~ 0
+Text Notes 9550 1000 0    80   ~ 0
 Bessel Bandpass Filter
-Text Notes 9550 850  0    50   ~ 0
-Measured loss of 4.5dB at 100MHz
-Text Notes 8150 700  0    50   ~ 0
-Buffer output is\n3.3Vp-p = 14.35dBm\nAfter Attenuator and Filter\nthe LO Level is about 7dBm\naccounting for component variation\n14.35dBm-2-4.5=7.85dBm
 Text Label 5100 3050 2    40   ~ 0
 RF
